File: Serial-Knob.kicad_pcb (KiCad board)
At the start: 2 copper layers, 23.5 x 23.5 mm, 15 parts, among them IC1 ATTINY85-S, P1 CONN_4

Commit message: Fixed missing module definitions (pcbnew BZR 4319 was barfing).
Parts:
- G1: value LOGO -> OSHW_LOGO; footprint (none) -> OSHW_LOGO
- G2: value LOGO -> LED_SMILE; footprint LOGO -> LED_SMILE
- G3: value Tindie -> TINDIE_DOG; footprint LOGO -> TINDIE_DOG
Changed lines of the file:
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@@
-(kicad_pcb (version 3) (host pcbnew "(2013-06-27 BZR 4227)-testing")
+(kicad_pcb (version 3) (host pcbnew "(2013-09-16 BZR 4319)-product")
   (general
     (links 30)
@@
     (pad_to_mask_clearance 0)
     (aux_axis_origin 0 0)
-    (visible_elements 7FFFFFBF)
+    (visible_elements 7FFFFF3F)
     (pcbplotparams
       (layerselection 317751297)
@@
     )
   )
-  (module LOGO (layer Front)
+  (module TINDIE_DOG (layer Front)
     (at 102.75 98.425)
     (fp_text reference G3 (at 0 1.43764) (layer F.SilkS) hide
       (effects (font (size 1 1) (thickness 0.2)))
     )
-    (fp_text value Tindie (at 0 -1.43764) (layer F.SilkS) hide
+    (fp_text value TINDIE_DOG (at 0 -1.43764) (layer F.SilkS) hide
       (effects (font (size 1 1) (thickness 0.2)))
     )
@@
       (xy 0.05334 -0.78232) (xy 0.05588 -0.77216) (xy 0.05588 -0.77216)) (layer F.Mask) (width 0.00254))
   )
-  (module MADW__SIL-4   locked (layer Front)
+  (module MADW__SIL-4 locked (layer Front)
     (at 113 87 180)
     (descr "Connecteur 4 pibs")
@@
     )
   )
-  (module LOGO (layer Front)
+  (module LED_SMILE (layer Front)
     (at 122.55 101.65)
-    (path LOGO)
     (fp_text reference G2 (at 0 1.97104) (layer F.SilkS) hide
       (effects (font (size 1 1) (thickness 0.2)))
     )
-    (fp_text value LOGO (at 0 -1.97104) (layer F.SilkS) hide
+    (fp_text value LED_SMILE (at 0 -1.97104) (layer F.SilkS) hide
       (effects (font (size 1 1) (thickness 0.2)))
     )
@@
       (xy 0.56134 -0.65532) (xy 0.60452 -0.64262) (xy 0.6096 -0.64262) (xy 0.65278 -0.64008)) (layer F.SilkS) (width 0.00254))
   )
-  (module "" (layer Front)
+  (module OSHW_LOGO (layer Front)
     (at 103.45 101.65)
     (fp_text reference G1 (at 0 1.77038) (layer F.SilkS) hide
       (effects (font (size 1 1) (thickness 0.2)))
     )
-    (fp_text value LOGO (at 0 -1.77038) (layer F.SilkS) hide
-      (effects (font (size 1 1) (thickness 0.2)))
-    )
+    (fp_text value OSHW_LOGO (at 0 -1.77038) (layer F.SilkS) hide
+      (effects (font (size 1 1) (thickness 0.2)))
+    )
