File: Serial-Knob__4x4.kicad_pcb (KiCad board)
At the start: 2 copper layers, 49 x 49 mm, 68 parts, among them IC1 ATTINY85-S, P1 CONN_4

Commit message: Fixed missing module definitions (pcbnew BZR 4319 was barfing).
Parts:
- G1 (x4): value LOGO -> OSHW_LOGO; footprint (none) -> OSHW_LOGO
- G2 (x4): value LOGO -> LED_SMILE; footprint LOGO -> LED_SMILE
- G3 (x4): value Tindie -> TINDIE_DOG; footprint LOGO -> TINDIE_DOG
Changed lines of the file:
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@@
-(kicad_pcb (version 3) (host pcbnew "(2013-05-16 BZR 4153)-testing")
+(kicad_pcb (version 3) (host pcbnew "(2013-09-16 BZR 4319)-product")
   (general
     (links 165)
@@
     )
   )
-  (module LOGO (layer Front)
+  (module TINDIE_DOG (layer Front)
     (at 102.75 46.425)
     (fp_text reference G3 (at 0 1.43764) (layer F.SilkS) hide
       (effects (font (size 1 1) (thickness 0.2)))
     )
-    (fp_text value Tindie (at 0 -1.43764) (layer F.SilkS) hide
+    (fp_text value TINDIE_DOG (at 0 -1.43764) (layer F.SilkS) hide
       (effects (font (size 1 1) (thickness 0.2)))
     )
@@
       (xy 0.05334 -0.78232) (xy 0.05588 -0.77216) (xy 0.05588 -0.77216)) (layer F.Mask) (width 0.00254))
   )
-  (module MADW__SIL-4   locked (layer Front)
+  (module MADW__SIL-4 locked (layer Front)
     (at 113 35 180)
     (descr "Connecteur 4 pibs")
@@
     )
   )
-  (module LOGO (layer Front)
+  (module LED_SMILE (layer Front)
     (at 122.55 49.65)
-    (path LOGO)
     (fp_text reference G2 (at 0 1.97104) (layer F.SilkS) hide
       (effects (font (size 1 1) (thickness 0.2)))
     )
-    (fp_text value LOGO (at 0 -1.97104) (layer F.SilkS) hide
+    (fp_text value LED_SMILE (at 0 -1.97104) (layer F.SilkS) hide
       (effects (font (size 1 1) (thickness 0.2)))
     )
@@
       (xy 0.56134 -0.65532) (xy 0.60452 -0.64262) (xy 0.6096 -0.64262) (xy 0.65278 -0.64008)) (layer F.SilkS) (width 0.00254))
   )
-  (module "" (layer Front)
+  (module OSHW_LOGO (layer Front)
     (at 103.45 49.65)
     (fp_text reference G1 (at 0 1.77038) (layer F.SilkS) hide
       (effects (font (size 1 1) (thickness 0.2)))
     )
-    (fp_text value LOGO (at 0 -1.77038) (layer F.SilkS) hide
+    (fp_text value OSHW_LOGO (at 0 -1.77038) (layer F.SilkS) hide
       (effects (font (size 1 1) (thickness 0.2)))
     )
@@
     )
   )
-  (module "" (layer Front)
+  (module OSHW_LOGO (layer Front)
     (at 77.95 49.65)
     (fp_text reference G1 (at 0 1.77038) (layer F.SilkS) hide
       (effects (font (size 1 1) (thickness 0.2)))
     )
-    (fp_text value LOGO (at 0 -1.77038) (layer F.SilkS) hide
+    (fp_text value OSHW_LOGO (at 0 -1.77038) (layer F.SilkS) hide
       (effects (font (size 1 1) (thickness 0.2)))
     )
@@
       (xy -1.01092 1.4986)) (layer F.SilkS) (width 0.00254))
   )
-  (module LOGO (layer Front)
+  (module LED_SMILE (layer Front)
     (at 97.05 49.65)
-    (path LOGO)
     (fp_text reference G2 (at 0 1.97104) (layer F.SilkS) hide
       (effects (font (size 1 1) (thickness 0.2)))
     )
-    (fp_text value LOGO (at 0 -1.97104) (layer F.SilkS) hide
+    (fp_text value LED_SMILE (at 0 -1.97104) (layer F.SilkS) hide
       (effects (font (size 1 1) (thickness 0.2)))
     )
@@
     )
   )
-  (module MADW__SIL-4   locked (layer Front)
+  (module MADW__SIL-4 locked (layer Front)
     (at 87.5 35 180)
     (descr "Connecteur 4 pibs")
@@
     )
   )
-  (module LOGO (layer Front)
+  (module TINDIE_DOG (layer Front)
     (at 77.25 46.425)
     (fp_text reference G3 (at 0 1.43764) (layer F.SilkS) hide
       (effects (font (size 1 1) (thickness 0.2)))
     )
-    (fp_text value Tindie (at 0 -1.43764) (layer F.SilkS) hide
+    (fp_text value TINDIE_DOG (at 0 -1.43764) (layer F.SilkS) hide
       (effects (font (size 1 1) (thickness 0.2)))
     )
@@
     )
   )
-  (module LOGO (layer Front)
+  (module TINDIE_DOG (layer Front)
     (at 77.25 71.925)
     (fp_text reference G3 (at 0 1.43764) (layer F.SilkS) hide
       (effects (font (size 1 1) (thickness 0.2)))
     )
-    (fp_text value Tindie (at 0 -1.43764) (layer F.SilkS) hide
+    (fp_text value TINDIE_DOG (at 0 -1.43764) (layer F.SilkS) hide
       (effects (font (size 1 1) (thickness 0.2)))
     )
@@
       (xy 0.05334 -0.78232) (xy 0.05588 -0.77216) (xy 0.05588 -0.77216)) (layer F.Mask) (width 0.00254))
   )
-  (module MADW__SIL-4   locked (layer Front)
+  (module MADW__SIL-4 locked (layer Front)
     (at 87.5 60.5 180)
     (descr "Connecteur 4 pibs")
@@
     )
   )
-  (module LOGO (layer Front)
+  (module LED_SMILE (layer Front)
     (at 97.05 75.15)
-    (path LOGO)
     (fp_text reference G2 (at 0 1.97104) (layer F.SilkS) hide
       (effects (font (size 1 1) (thickness 0.2)))
     )
-    (fp_text value LOGO (at 0 -1.97104) (layer F.SilkS) hide
+    (fp_text value LED_SMILE (at 0 -1.97104) (layer F.SilkS) hide
       (effects (font (size 1 1) (thickness 0.2)))
     )
@@
       (xy 0.56134 -0.65532) (xy 0.60452 -0.64262) (xy 0.6096 -0.64262) (xy 0.65278 -0.64008)) (layer F.SilkS) (width 0.00254))
   )
-  (module "" (layer Front)
+  (module OSHW_LOGO (layer Front)
     (at 77.95 75.15)
     (fp_text reference G1 (at 0 1.77038) (layer F.SilkS) hide
       (effects (font (size 1 1) (thickness 0.2)))
     )
-    (fp_text value LOGO (at 0 -1.77038) (layer F.SilkS) hide
+    (fp_text value OSHW_LOGO (at 0 -1.77038) (layer F.SilkS) hide
       (effects (font (size 1 1) (thickness 0.2)))
     )
@@
     )
   )
-  (module "" (layer Front)
+  (module OSHW_LOGO (layer Front)
     (at 103.45 75.15)
     (fp_text reference G1 (at 0 1.77038) (layer F.SilkS) hide
       (effects (font (size 1 1) (thickness 0.2)))
     )
-    (fp_text value LOGO (at 0 -1.77038) (layer F.SilkS) hide
+    (fp_text value OSHW_LOGO (at 0 -1.77038) (layer F.SilkS) hide
       (effects (font (size 1 1) (thickness 0.2)))
     )
@@
       (xy -1.01092 1.4986)) (layer F.SilkS) (width 0.00254))
   )
-  (module LOGO (layer Front)
+  (module LED_SMILE (layer Front)
     (at 122.55 75.15)
-    (path LOGO)
     (fp_text reference G2 (at 0 1.97104) (layer F.SilkS) hide
       (effects (font (size 1 1) (thickness 0.2)))
     )
-    (fp_text value LOGO (at 0 -1.97104) (layer F.SilkS) hide
+    (fp_text value LED_SMILE (at 0 -1.97104) (layer F.SilkS) hide
       (effects (font (size 1 1) (thickness 0.2)))
     )
@@
     )
   )
-  (module MADW__SIL-4   locked (layer Front)
+  (module MADW__SIL-4 locked (layer Front)
     (at 113 60.5 180)
     (descr "Connecteur 4 pibs")
@@
     )
   )
-  (module LOGO (layer Front)
+  (module TINDIE_DOG (layer Front)
     (at 102.75 71.925)
     (fp_text reference G3 (at 0 1.43764) (layer F.SilkS) hide
       (effects (font (size 1 1) (thickness 0.2)))
     )
-    (fp_text value Tindie (at 0 -1.43764) (layer F.SilkS) hide
+    (fp_text value TINDIE_DOG (at 0 -1.43764) (layer F.SilkS) hide
       (effects (font (size 1 1) (thickness 0.2)))
     )
